File: kicad/pulsar.sch (KiCad schematic (older format))
At the start: 51 parts, among them J1 POWER, J2 JTAG, J3 XO2-JTAG, J4 CONN-2x5, U1 TS1102, U2 XO2-256, U3 MIC5205, U4 nrf51822, Y1 32kHz, Y2 16MHz

Commit message: start layout
Parts:
- D1, D2, D3: footprint SMD-1005:SMD-1005 -> libs:SMD-1608-LED
- J2: value JTAG -> NRF-SWD; footprint (none) -> libs:CONN-2x5-1.27-SMT
- J3, J4: footprint (none) -> libs:CONN-2x5-1.27-SMT
- R4, R5, R6, R7, RT1: footprint SMD-1608:SMD-1608 -> SMD-1005:SMD-1005
- Y2: symbol XTAL -> XTAL-4
Changed lines of the file:
@@
 $EndComp
 $Comp
-L XTAL Y2
+L XTAL-4 Y2
 U 1 1 54134AE5
 P 7950 2500
@@
 F 3 "" H 7950 2500 60  0000 C CNN
 	1    7950 2500
-	1    0    0    1
+	1    0    0    -1
 $EndComp
 $Comp
@@
 Text Label 6300 1800 2    50   ~ 0
 SPI_CS
-Text Label 6300 1200 2    50   ~ 0
+Text Label 5850 3150 2    50   ~ 0
 ~XO2_JTAG_EN
 Text Label 6300 1300 2    50   ~ 0
@@
 Text Label 6300 1000 2    50   ~ 0
 XO2_JTAG_TDO
-Text Label 6300 1100 2    50   ~ 0
+Text Label 5850 3050 2    50   ~ 0
 ~XO2_RESET
 $Comp
@@
 F 0 "RT1" H 1675 3805 30  0000 L CNN
 F 1 "47k" H 1675 3755 30  0000 L CNN
-F 2 "SMD-1608:SMD-1608" H 1650 3750 60  0001 C CNN
+F 2 "SMD-1005:SMD-1005" H 1650 3750 60  0001 C CNN
 F 3 "" H 1650 3750 60  0000 C CNN
 	1    1650 3750
@@
 F 0 "R4" H 1675 3575 30  0000 L CNN
 F 1 "22k" H 1675 3525 30  0000 L CNN
-F 2 "SMD-1608:SMD-1608" H 1650 3550 60  0001 C CNN
+F 2 "SMD-1005:SMD-1005" H 1650 3550 60  0001 C CNN
 F 3 "" H 1650 3550 60  0000 C CNN
 	1    1650 3550
@@
 Wire Wire Line
 	8200 2400 8200 2450
-Wire Wire Line
-	8200 2450 8250 2450
 Connection ~ 7950 2400
 Wire Wire Line
-	8250 2550 8200 2550
-Wire Wire Line
-	8200 2550 8200 2600
+	8200 2600 8200 2550
 Connection ~ 7950 2600
 Wire Wire Line
@@
 	5400 4150 4750 4150
 Wire Wire Line
-	5550 1200 6300 1200
+	5100 3150 5850 3150
 Wire Wire Line
 	5550 1300 6300 1300
@@
 	5550 1000 6300 1000
 Wire Wire Line
-	5550 1100 6300 1100
+	5100 3050 5850 3050
 Wire Wire Line
 	6300 1600 5550 1600
@@
 F 0 "D1" H 6175 4425 30  0000 L CNN
 F 1 "LED" H 6175 4375 30  0000 L CNN
-F 2 "SMD-1005:SMD-1005" H 6150 4400 60  0001 C CNN
+F 2 "libs:SMD-1608-LED" H 6150 4400 60  0001 C CNN
 F 3 "" H 6150 4400 60  0000 C CNN
 	1    6150 4400
@@
 F 0 "D2" H 6375 4425 30  0000 L CNN
 F 1 "LED" H 6375 4375 30  0000 L CNN
-F 2 "SMD-1005:SMD-1005" H 6350 4400 60  0001 C CNN
+F 2 "libs:SMD-1608-LED" H 6350 4400 60  0001 C CNN
 F 3 "" H 6350 4400 60  0000 C CNN
 	1    6350 4400
@@
 F 0 "D3" H 6575 4425 30  0000 L CNN
 F 1 "LED" H 6575 4375 30  0000 L CNN
-F 2 "SMD-1005:SMD-1005" H 6550 4400 60  0001 C CNN
+F 2 "libs:SMD-1608-LED" H 6550 4400 60  0001 C CNN
 F 3 "" H 6550 4400 60  0000 C CNN
 	1    6550 4400
@@
 F 0 "R5" H 6175 4225 30  0000 L CNN
 F 1 "1k" H 6175 4175 30  0000 L CNN
-F 2 "SMD-1608:SMD-1608" H 6150 4200 60  0001 C CNN
+F 2 "SMD-1005:SMD-1005" H 6150 4200 60  0001 C CNN
 F 3 "" H 6150 4200 60  0000 C CNN
 	1    6150 4200
@@
 F 0 "R6" H 6375 4225 30  0000 L CNN
 F 1 "1k" H 6375 4175 30  0000 L CNN
-F 2 "SMD-1608:SMD-1608" H 6350 4200 60  0001 C CNN
+F 2 "SMD-1005:SMD-1005" H 6350 4200 60  0001 C CNN
 F 3 "" H 6350 4200 60  0000 C CNN
 	1    6350 4200
@@
 F 0 "R7" H 6575 4225 30  0000 L CNN
 F 1 "1k" H 6575 4175 30  0000 L CNN
-F 2 "SMD-1608:SMD-1608" H 6550 4200 60  0001 C CNN
+F 2 "SMD-1005:SMD-1005" H 6550 4200 60  0001 C CNN
 F 3 "" H 6550 4200 60  0000 C CNN
 	1    6550 4200
@@
 P 9400 4250
 F 0 "J2" H 9000 3900 50  0000 L CNN
-F 1 "JTAG" H 9800 3900 50  0000 R CNN
-F 2 "" H 9300 4050 50  0001 C CNN
+F 1 "NRF-SWD" H 9800 3900 50  0000 R CNN
+F 2 "libs:CONN-2x5-1.27-SMT" H 9300 4050 50  0001 C CNN
 F 3 "" H 9300 4050 50  0000 C CNN
 	1    9400 4250
@@
 F 0 "J3" H 9000 4750 50  0000 L CNN
 F 1 "XO2-JTAG" H 9800 4750 50  0000 R CNN
-F 2 "" H 9300 4900 50  0001 C CNN
+F 2 "libs:CONN-2x5-1.27-SMT" H 9300 4900 50  0001 C CNN
 F 3 "" H 9300 4900 50  0000 C CNN
 	1    9400 5100
@@
 F 0 "J4" H 9400 5700 50  0000 C CNN
 F 1 "CONN-2x5" H 9400 5600 50  0000 C CNN
-F 2 "" H 10000 6800 50  0001 C CNN
+F 2 "libs:CONN-2x5-1.27-SMT" H 10000 6800 50  0001 C CNN
 F 3 "" H 10000 6800 50  0000 C CNN
 	1    9400 6000
@@
 $EndComp
 Wire Wire Line
-	4550 1500 4100 1500
-Text Label 4100 1500 0    50   ~ 0
+	4550 1000 4100 1000
+Text Label 4100 1000 0    50   ~ 0
 AUX1
 Wire Wire Line
-	4100 1600 4550 1600
-Wire Wire Line
-	4550 1700 4100 1700
-Wire Wire Line
-	4100 1800 4550 1800
-Wire Wire Line
-	4550 1900 4100 1900
-Text Label 4100 1600 0    50   ~ 0
+	4100 1100 4550 1100
+Wire Wire Line
+	5550 2200 6000 2200
+Wire Wire Line
+	6000 2300 5550 2300
+Wire Wire Line
+	5550 2400 6000 2400
+Text Label 4100 1100 0    50   ~ 0
 AUX2
-Text Label 4100 1700 0    50   ~ 0
+Text Label 6000 2200 2    50   ~ 0
 AUX3
-Text Label 4100 1800 0    50   ~ 0
+Text Label 6000 2300 2    50   ~ 0
 AUX4
-Text Label 4100 1900 0    50   ~ 0
+Text Label 6000 2400 2    50   ~ 0
 AUX5
 Wire Wire Line
@@
 AUX5
 Wire Wire Line
-	5550 2300 6100 2300
-Text Label 6100 2400 2    50   ~ 0
+	5550 1100 6100 1100
+Text Label 6100 1200 2    50   ~ 0
 RX
 Wire Wire Line
-	6100 2400 5550 2400
-Text Label 6100 2300 2    50   ~ 0
+	6100 1200 5550 1200
+Text Label 6100 1100 2    50   ~ 0
 TX
 Wire Wire Line
@@
 Wire Wire Line
 	6800 1950 6800 2150
-NoConn ~ 4550 1000
-NoConn ~ 4550 1100
+NoConn ~ 4550 1900
+NoConn ~ 4550 1800
 NoConn ~ 4550 2200
-NoConn ~ 5550 2200
+NoConn ~ 4550 1700
 $Comp
 L POWER_FLAG #PWR049
@@
 $EndComp
 Connection ~ 1000 2100
+Wire Wire Line
+	7850 2450 7850 2550
+Wire Wire Line
+	7850 2450 7650 2450
+Connection ~ 7650 2450
 $EndSCHEMATC

Commit message: more layouting
Parts:
- added C26: 1u, SMD-1005:SMD-1005, symbol C
- AE1: footprint (none) -> libs:ANT3216
- B1: footprint (none) -> libs:BALUN-2450BM14E0003
- C1: value 1u -> 10u
- C12, C13, C14, C2, C3, C4, C7, C8: value C -> 100n
- C15, C5: value C -> 1u
- C16, C17: value 12pF -> 7p
- C18, C21, C24: value 100nF -> 100n
- C19, C20: value 12pF -> 6p
- C22: value 47nF -> 47n
- C23: value 2.2nF -> 2.2n
- C25: value 1nF -> 1n
- C6: value 2.2u -> 4.7u
- J1: footprint (none) -> libs:TERM-2-3.5-PTH
- S1, S2: footprint (none) -> libs:TACT-4632
- Y1: footprint (none) -> libs:OSC2012
- Y2: value 16MHz -> 32MHz; footprint osc2520:OSC2520 -> libs:OSC2016
Connections:
- wire segments 232 -> 231
- no-connect marks 10 -> 12
Other:
- moved on the sheet: C15, C18, C19, C20, C24, C3, C5

Commit message: layout progress
Parts:
- added MH1, MH2, MH3, MH4: MOUNTHOLE, libs:HOLE-M3-COND, symbol MOUNTHOLE
- C1: footprint SMD-1005:SMD-1005 -> SMD-2012:SMD-2012
- R1, R2: footprint SMD-1608:SMD-1608 -> SMD-1005:SMD-1005
Connections:
- net labels removed: AUX5
- no-connect marks 12 -> 13
Other:
- moved on the sheet: C11, C5, C9

Commit message: more layout
Connections:
- net labels added: SPI_CS_PGM
- wire segments 231 -> 270
- no-connect marks 13 -> 20
Other:
- moved on the sheet: C10, C11, C14, C15, C2, C4, C5, C9

Commit message: layout
Connections:
- wire segments 270 -> 226
- no-connect marks 20 -> 18
Changed lines of the file:
@@
 Text Label 800  5800 0    50   ~ 0
 XO2_JTAG_TDO
-Text Label 4200 6800 2    50   ~ 0
+Text Label 4200 5800 2    50   ~ 0
 CH10
-Text Label 4200 6900 2    50   ~ 0
+Text Label 4200 6200 2    50   ~ 0
 CH11
 Text Label 1150 5900 0    50   ~ 0
@@
 Text Label 800  6000 0    50   ~ 0
 ~XO2_RESET
-Text Label 4200 5800 2    50   ~ 0
+Text Label 4200 6300 2    50   ~ 0
 CH12
+Text Label 4200 6900 2    50   ~ 0
+CH9
+Text Label 550  6600 0    50   ~ 0
+CH6
 Text Label 550  5800 0    50   ~ 0
-CH9
-Text Label 550  6400 0    50   ~ 0
-CH6
-Text Label 550  6500 0    50   ~ 0
 CH7
-Text Label 550  6600 0    50   ~ 0
+Text Label 4200 6800 2    50   ~ 0
 CH8
 Text Label 1150 6800 0    50   ~ 0
@@
 Text Label 7350 2200 0    50   ~ 0
 NRF_SWDIO/~RESET
-NoConn ~ 4750 4250
-Text Label 5400 4150 2    50   ~ 0
+NoConn ~ 4750 4150
+Text Label 5400 4250 2    50   ~ 0
 BUTTON2
 Text Label 6300 1900 2    50   ~ 0
@@
 	1    0    0    -1
 $EndComp
+Text Label 3600 1400 0    50   ~ 0
+VIN_SENSE
 Text Label 3600 1300 0    50   ~ 0
-VIN_SENSE
-Text Label 3600 1400 0    50   ~ 0
 IIN_SENSE
 $Comp
@@
 	9200 2450 9500 2450
 Wire Wire Line
-	9200 2550 9400 2550
-Wire Wire Line
-	9400 2550 9500 2550
+	9200 2550 9500 2550
 Wire Wire Line
 	9400 2650 9400 2550
@@
 	10400 2550 10500 2550
 Wire Wire Line
-	10500 2450 10500 2550
-Wire Wire Line
-	10500 2550 10500 2750
+	10500 2450 10500 2750
 Wire Wire Line
 	10400 2450 10500 2450
@@
 	10400 2350 10750 2350
 Wire Wire Line
-	7500 1300 7600 1300
-Wire Wire Line
-	7600 1300 7750 1300
-Wire Wire Line
-	7750 1300 7900 1300
-Wire Wire Line
-	7900 1300 8150 1300
-Wire Wire Line
-	8150 1300 8200 1300
+	7500 1300 8200 1300
 Wire Wire Line
 	9800 1450 9800 1350
 Wire Wire Line
-	9200 1450 9250 1450
-Wire Wire Line
-	9250 1450 9700 1450
-Wire Wire Line
-	9700 1450 9800 1450
+	9200 1450 9800 1450
 Wire Wire Line
 	9200 1550 9250 1550
@@
 	7600 2600 7700 2600
 Wire Wire Line
-	7800 2600 7950 2600
-Wire Wire Line
-	7950 2600 8200 2600
-Wire Wire Line
-	7800 2400 7950 2400
-Wire Wire Line
-	7950 2400 8200 2400
+	7800 2600 8200 2600
+Wire Wire Line
+	7800 2400 8200 2400
 Wire Wire Line
 	8200 2400 8200 2450
@@
 	8200 1550 8100 1550
 Wire Wire Line
-	8100 1550 8100 1650
-Wire Wire Line
-	8100 1650 8100 1750
-Wire Wire Line
-	8100 1750 8100 1850
-Wire Wire Line
-	8100 1850 8100 1900
+	8100 1550 8100 1900
 Wire Wire Line
 	8100 1850 8200 1850
@@
 	7750 1500 7750 1450
 Wire Wire Line
-	7500 1500 7600 1500
-Wire Wire Line
-	7600 1500 7750 1500
-Wire Wire Line
-	7750 1500 7900 1500
+	7500 1500 7900 1500
 Wire Wire Line
 	7900 1500 7900 1450
@@
 	2600 7250 2600 7350
 Wire Wire Line
-	2600 7350 2700 7350
-Wire Wire Line
-	2700 7350 2800 7350
+	2600 7350 2800 7350
 Wire Wire Line
 	2700 7350 2700 7250
@@
 	1350 2200 1350 2100
 Wire Wire Line
-	950  2100 1000 2100
-Wire Wire Line
-	1000 2100 1100 2100
-Wire Wire Line
-	1100 2100 1350 2100
-Wire Wire Line
-	1350 2100 1400 2100
+	950  2100 1400 2100
 Connection ~ 1350 2100
 Wire Wire Line
@@
 	1100 2250 1100 2300
 Wire Wire Line
-	2100 2100 2250 2100
-Wire Wire Line
-	2250 2100 2450 2100
+	2100 2100 2450 2100
 Wire Wire Line
 	2250 2100 2250 2150
@@
 	1050 850  1200 850
 Wire Wire Line
-	1200 850  1200 1100
-Wire Wire Line
-	1200 1100 1200 1200
-Wire Wire Line
-	1700 750  2100 750
-Wire Wire Line
-	2100 750  2350 750
+	1200 850  1200 1200
+Wire Wire Line
+	1700 750  2350 750
 Wire Wire Line
 	2350 750  2350 700
@@
 	3900 5700 3800 5700
 Wire Wire Line
-	3900 5300 3900 5600
-Wire Wire Line
-	3900 5600 3900 5700
+	3900 5300 3900 5700
 Connection ~ 3900 5600
 Wire Wire Line
@@
 Connection ~ 4050 5300
 Wire Wire Line
-	3900 5300 4050 5300
-Wire Wire Line
-	4050 5300 4250 5300
-Wire Wire Line
-	4250 5300 4400 5300
+	3900 5300 4400 5300
 Wire Wire Line
 	4050 5450 4050 5500
 Wire Wire Line
-	4050 5500 4250 5500
-Wire Wire Line
-	4250 5500 4400 5500
+	4050 5500 4400 5500
 Wire Wire Line
 	3200 4950 3200 4900
@@
 Connection ~ 2900 4950
 Wire Wire Line
-	2750 4950 2900 4950
-Wire Wire Line
-	2900 4950 3050 4950
-Wire Wire Line
-	3050 4950 3200 4950
+	2750 4950 3200 4950
 Wire Wire Line
 	3050 4950 3050 5000
@@
 	2900 5100 2900 5150
 Wire Wire Line
-	2900 5150 3050 5150
-Wire Wire Line
-	3050 5150 3200 5150
+	2900 5150 3200 5150
 Wire Wire Line
 	3050 5150 3050 5100
 Connection ~ 3050 5150
 Wire Wire Line
-	2750 4950 2750 5300
-Wire Wire Line
-	2750 5300 2750 5350
+	2750 4950 2750 5350
 Wire Wire Line
 	2650 5350 2650 5300
@@
 Connection ~ 1300 5300
 Wire Wire Line
-	650  5300 800  5300
-Wire Wire Line
-	800  5300 1000 5300
-Wire Wire Line
-	1000 5300 1150 5300
-Wire Wire Line
-	1150 5300 1300 5300
-Wire Wire Line
-	1300 5300 1450 5300
+	650  5300 1450 5300
 Wire Wire Line
 	1000 5300 1000 5350
@@
 	1300 5500 1300 5450
 Wire Wire Line
-	650  5500 800  5500
-Wire Wire Line
-	800  5500 1000 5500
-Wire Wire Line
-	1000 5500 1150 5500
-Wire Wire Line
-	1150 5500 1300 5500
+	650  5500 1300 5500
 Wire Wire Line
 	1000 5500 1000 5450
 Connection ~ 1000 5500
 Wire Wire Line
-	1450 5300 1450 5600
-Wire Wire Line
-	1450 5600 1450 5700
+	1450 5300 1450 5700
 Wire Wire Line
 	1450 5700 1550 5700
@@
 	1550 6100 800  6100
 Wire Wire Line
-	550  6400 1550 6400
-Wire Wire Line
-	550  6500 1550 6500
+	800  6400 1550 6400
+Wire Wire Line
+	800  6500 1550 6500
 Wire Wire Line
 	550  6600 1550 6600
@@
 Connection ~ 4050 7200
 Wire Wire Line
-	3900 7200 4050 7200
-Wire Wire Line
-	4050 7200 4200 7200
+	3900 7200 4200 7200
 Wire Wire Line
 	4050 7350 4050 7400
@@
 	1200 7200 1200 7150
 Wire Wire Line
-	1200 7200 1350 7200
-Wire Wire Line
-	1350 7200 1450 7200
+	1200 7200 1450 7200
 Wire Wire Line
 	1350 7200 1350 7250
@@
 	7350 2200 8200 2200
 Wire Wire Line
-	4350 4150 4350 4250
-Wire Wire Line
-	4350 4250 4350 4300
+	4350 4150 4350 4300
 Connection ~ 4350 4250
 Wire Wire Line
-	5400 4150 4750 4150
+	5400 4250 4750 4250
 Wire Wire Line
 	5550 2200 6100 2200
@@
 	-1   0    0    -1
 $EndComp
-NoConn ~ 4750 3750
-Text Label 5400 3650 2    50   ~ 0
+NoConn ~ 4750 3650
+Text Label 5400 3750 2    50   ~ 0
 BUTTON1
 Wire Wire Line
-	4350 3650 4350 3750
-Wire Wire Line
-	4350 3750 4350 3800
+	4350 3650 4350 3800
 Connection ~ 4350 3750
 Wire Wire Line
-	5400 3650 4750 3650
+	5400 3750 4750 3750
 $Comp
 L DGND #PWR042
@@
 	8600 5000 8800 5000
 Wire Wire Line
-	8600 5000 8600 5050
-Wire Wire Line
-	8600 5050 8600 5100
+	8600 5000 8600 5100
 Wire Wire Line
 	8600 5100 8800 5100
@@
 	8600 4150 8800 4150
 Wire Wire Line
-	8600 4150 8600 4200
-Wire Wire Line
-	8600 4200 8600 4250
+	8600 4150 8600 4250
 Wire Wire Line
 	8600 4250 8800 4250
@@
 	6800 2150 6700 2150
 Wire Wire Line
-	6250 2150 6500 2150
-Wire Wire Line
-	6500 2150 6600 2150
-Wire Wire Line
-	6250 1950 6500 1950
-Wire Wire Line
-	6500 1950 6600 1950
+	6250 2150 6600 2150
+Wire Wire Line
+	6250 1950 6600 1950
 Connection ~ 6500 1950
 Connection ~ 6500 2150
@@
 	1    0    0    -1
 $EndComp
-NoConn ~ 3800 6100
-NoConn ~ 3800 6200
-NoConn ~ 3800 6300
+NoConn ~ 3800 6400
 Wire Wire Line
 	1150 5350 1150 5300
@@
 NoConn ~ 5550 1000
 Wire Wire Line
-	3800 6400 4350 6400
-Text Label 4350 6400 2    50   ~ 0
+	3800 6100 4350 6100
+Text Label 4350 6100 2    50   ~ 0
 SPI_CS
 Wire Wire Line
@@
 Text Label 6300 1600 2    50   ~ 0
 SPI_CS_PGM
+Wire Wire Line
+	3800 6200 4200 6200
+Wire Wire Line
+	3800 6300 4200 6300
 $EndSCHEMATC

Commit message: switch to 4 layers
Other:
- note added: "XXX test point for SPI_PGM_CS"
Changed lines of the file:
@@
 Wire Wire Line
 	3800 6300 4200 6300
+Text Notes 4100 3300 0    50   ~ 0
+XXX test point for SPI_PGM_CS
 $EndSCHEMATC

Commit message: layout work
Connections:
- net labels added: RAW_VIN
Other:
- note added: "XXX inductor?"
Changed lines of the file:
@@
 Text Notes 4100 3300 0    50   ~ 0
 XXX test point for SPI_PGM_CS
+Text Notes 550  2300 0    50   ~ 0
+XXX inductor?
+Text Label 1100 750  0    50   ~ 0
+RAW_VIN
 $EndSCHEMATC

Commit message: layout changes
Parts:
- added TP1: PGM, libs:TESTPOINT-1.0, symbol TESTPOINT
- FB1: footprint SMD-1005:SMD-1005 -> SMD-2012:SMD-2012
Connections:
- wire segments 226 -> 228
Other:
- note removed: "XXX test point for SPI_PGM_CS"
Changed lines of the file:
@@
 EESchema Schematic File Version 2
+LIBS:testpoint
 LIBS:mounthole
 LIBS:power_flag
@@
 F 0 "FB1" H 775 2025 40  0000 L CNN
 F 1 "FERRITE" H 850 2200 60  0001 C CNN
-F 2 "SMD-1005:SMD-1005" H 850 2000 60  0001 C CNN
+F 2 "SMD-2012:SMD-2012" H 850 2000 60  0001 C CNN
 F 3 "" H 850 2000 60  0000 C CNN
 	1    850  2100
@@
 Wire Wire Line
 	3800 6300 4200 6300
-Text Notes 4100 3300 0    50   ~ 0
-XXX test point for SPI_PGM_CS
 Text Notes 550  2300 0    50   ~ 0
 XXX inductor?
 Text Label 1100 750  0    50   ~ 0
 RAW_VIN
+$Comp
+L TESTPOINT TP1
+U 1 1 5454B95A
+P 8250 5950
+F 0 "TP1" H 8325 6000 30  0000 C CNN
+F 1 "PGM" H 8250 6125 30  0000 C CNN
+F 2 "libs:TESTPOINT-1.0" H 8250 5950 50  0001 C CNN
+F 3 "" H 8250 5950 50  0000 C CNN
+	1    8250 5950
+	1    0    0    -1
+$EndComp
+Wire Wire Line
+	8250 5950 8250 6050
+Wire Wire Line
+	8250 6050 7600 6050
+Text Label 7600 6050 0    50   ~ 0
+SPI_CS_PGM
 $EndSCHEMATC
