File: kicad/pulsar.sch (KiCad schematic (older format))
At the start: 57 parts, among them J1 POWER, J2 NRF-SWD, J3 XO2-JTAG, J4 CONN-2x5, U1 TS1102, U2 XO2-256, U3 MIC5205, U4 nrf51822, Y1 32kHz, Y2 32MHz

Commit message: update component values, bring out values on assembly layer
Parts:
- C16, C17: value 7p -> 20p
- C19, C20: value 6p -> 7p
- C25: value 1n -> 2.2n
- R1: value 190k -> 124k
- U1: value TS1102 -> TS1102-50
Changed lines of the file:
@@
 P 7750 2600
 F 0 "C20" H 7775 2625 30  0000 L CNN
-F 1 "6p" H 7775 2575 30  0000 L CNN
+F 1 "7p" H 7775 2575 30  0000 L CNN
 F 2 "SMD-1005:SMD-1005" H 7650 2650 60  0001 C CNN
 F 3 "" H 7650 2650 60  0000 C CNN
@@
 P 7750 2400
 F 0 "C19" H 7775 2425 30  0000 L CNN
-F 1 "6p" H 7775 2375 30  0000 L CNN
+F 1 "7p" H 7775 2375 30  0000 L CNN
 F 2 "SMD-1005:SMD-1005" H 7650 2450 60  0001 C CNN
 F 3 "" H 7650 2450 60  0000 C CNN
@@
 P 9700 1550
 F 0 "C25" H 9725 1575 30  0000 L CNN
-F 1 "1n" H 9725 1525 30  0000 L CNN
+F 1 "2.2n" H 9725 1525 30  0000 L CNN
 F 2 "SMD-1005:SMD-1005" H 9600 1600 60  0001 C CNN
 F 3 "" H 9600 1600 60  0000 C CNN
@@
 P 700 3600
 F 0 "R1" H 725 3625 30  0000 L CNN
-F 1 "190k" H 725 3575 30  0000 L CNN
+F 1 "124k" H 725 3575 30  0000 L CNN
 F 2 "SMD-1005:SMD-1005" H 700 3600 60  0001 C CNN
 F 3 "" H 700 3600 60  0000 C CNN
@@
 P 1400 900
 F 0 "U1" H 1800 450 50  0000 R CNN
-F 1 "TS1102" H 1600 350 50  0000 L CNN
+F 1 "TS1102-50" H 1600 350 50  0000 L CNN
 F 2 "sot-23-5:SOT-23-5" H 950 1050 50  0001 C CNN
 F 3 "" H 950 1050 50  0000 C CNN
@@
 P 6650 2150
 F 0 "C17" H 6675 2175 30  0000 L CNN
-F 1 "7p" H 6675 2125 30  0000 L CNN
+F 1 "20p" H 6675 2125 30  0000 L CNN
 F 2 "SMD-1005:SMD-1005" H 6550 2200 60  0001 C CNN
 F 3 "" H 6550 2200 60  0000 C CNN
@@
 P 6650 1950
 F 0 "C16" H 6675 1975 30  0000 L CNN
-F 1 "7p" H 6675 1925 30  0000 L CNN
+F 1 "20p" H 6675 1925 30  0000 L CNN
 F 2 "SMD-1005:SMD-1005" H 6550 2000 60  0001 C CNN
 F 3 "" H 6550 2000 60  0000 C CNN
