File: kicad/pulsar.kicad_pcb (KiCad board)
At the start: 4 copper layers, 50 x 50 mm, 76 parts, among them J1 POWER, J13 CONN-2, J14 CONN-2, J15 CONN-2, J16 CONN-2, J2 NRF-SWD, J3 XO2-JTAG, J4 CONN-2x5, J5 CONN-4, J6 CONN-4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

Commit message: layout work
Connections:
- net Net-(J1-Pad1) renamed /RAW_VIN
Routing:
- net VIN: track 26.1 -> 39.0 mm, vias 0 -> 9
- net DGND: track 343.5 -> 346.5 mm, vias 182 -> 184
- added copper zone on F.Cu, net /RAW_VIN

Commit message: layout finish
Routing:
- net DGND: track 346.5 -> 349.5 mm
Other:
- rule pad_to_mask_clearance: 0 -> 0.05

Commit message: layout tweaks
Routing:
- net (no net): track 0.94 -> 0.00 mm, vias 1 -> 0
Changed lines of the file:
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@@
     (thickness 1.6)
     (drawings 7)
-    (tracks 1095)
+    (tracks 1092)
     (zones 0)
     (modules 76)
@@
   (module SMD-1005:SMD-1005 (layer F.Cu)
     (at 112.75 120 180)
-    (fp_text reference C18 (at 0 2 270) (layer F.SilkS)
+    (fp_text reference C18 (at 0.25 2 270) (layer F.SilkS)
       (effects (font (size 0.7 0.7) (thickness 0.15)))
     )
@@
   (module SMD-1005:SMD-1005 (layer F.Cu)
     (at 113.75 120 180)
-    (fp_text reference C26 (at 0 2 270) (layer F.SilkS)
+    (fp_text reference C26 (at -1 0 270) (layer F.SilkS)
       (effects (font (size 0.7 0.7) (thickness 0.15)))
     )
@@
   (gr_line (start 150 150) (end 100 150) (angle 90) (layer Edge.Cuts) (width 0.2))
   (gr_line (start 150 100) (end 150 150) (angle 90) (layer Edge.Cuts) (width 0.2))
-  (segment (start 111.900198 117.500198) (end 111.8 117.4) (width 0.129) (layer F.Cu) (net 0))
-  (via (at 111.8 117.4) (size 0.46) (layers F.Cu B.Cu) (net 0))
-  (segment (start 111.900198 117.500198) (end 111.900198 118.300198) (width 0.129) (layer F.Cu) (net 0))
   (segment (start 105.85 102.05) (end 105.2 102.05) (width 0.129) (layer F.Cu) (net 1) (status 10))
   (segment (start 105.2 103.95) (end 105.85 103.95) (width 0.129) (layer F.Cu) (net 1) (status 20))
@@
   (segment (start 128 106) (end 128 103.81) (width 0.5) (layer F.Cu) (net 62) (status 10))
   (segment (start 128 103.81) (end 127.19 103) (width 0.5) (layer F.Cu) (net 62) (status 20))
-  (segment (start 110.9 128.5) (end 110.9 129.22) (width 0.2) (layer F.Cu) (net 63) (status 400000))
+  (segment (start 110.9 128.5) (end 110.9 129.22) (width 0.2) (layer F.Cu) (net 63))
   (segment (start 110.9 129.22) (end 110.83 129.29) (width 0.2) (layer F.Cu) (net 63))
-  (segment (start 110.5 128.5) (end 110.5 129.11) (width 0.2) (layer F.Cu) (net 63) (status 400000))
+  (segment (start 110.5 128.5) (end 110.5 129.11) (width 0.2) (layer F.Cu) (net 63))
   (segment (start 110.5 129.11) (end 110.59 129.2) (width 0.2) (layer F.Cu) (net 63))
   (segment (start 117.5 107.5) (end 117.5 110) (width 0.129) (layer F.Cu) (net 63))

Commit message: layout changes
Parts:
- added TP1: PGM, libs:TESTPOINT-1.0, F.Cu at (121.8, 126.2)
- FB1: footprint SMD-1005:SMD-1005 -> SMD-2012:SMD-2012
- moved C1 1.46 mm to (108.5, 104.2), turned to 90 degrees
- moved FB1 1.03 mm to (108.5, 102.2), turned to 270 degrees
- moved R1 1.00 mm to (109.0, 106.8)
- moved R2 1.00 mm to (109.0, 107.8)
Connections:
- net DGND renamed PGND
Routing:
- net PGND: track 349.5 -> 351.3 mm, vias 184 -> 185
- net /SPI_CS_PGM: track 13.8 -> 15.0 mm
- net /VIN_SENSE: track 18.2 -> 17.3 mm
- net /IIN_SENSE: track 39.9 -> 40.5 mm

Commit message: add small logo
Other:
- board text added: "sternlabs .:.pulsar"
Changed lines of the file:
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@@
     (links 245)
     (no_connects 0)
-    (area 99.899999 99.899999 150.100001 150.100001)
+    (area 25.725 76.9 173 167.700001)
     (thickness 1.6)
-    (drawings 7)
+    (drawings 8)
     (tracks 1087)
     (zones 0)
@@
       (net 1 "Net-(C1-Pad1)"))
   )
+  (gr_text "sternlabs\n.:.pulsar" (at 120.75 115) (layer F.Mask)
+    (effects (font (size 1.5 1.5) (thickness 0.15)) (justify left))
+  )
   (gr_text "50R Antenna feed on FR-408 170um\ncoplanar wave guide with ground plane,\n260um conductor, 135um spacing\n(see antenna_waveguide_4l.xsctn)" (at 25.75 81.25) (layer Cmts.User)

Commit message: update component values, bring out values on assembly layer
Parts:
- C16, C17: value 7p -> 20p
- C19, C20: value 6p -> 7p
- C25: value 1n -> 2.2n
- R1: value 190k -> 124k
- U1: value TS1102 -> TS1102-50
